Commit message: deploy: fix ROS2 controller/plugin to the verified V14 contract
Per sim2sim measurements (official 13k policy, vx=1.0 -> 0.935 m/s):
- rl_controller: rear-first leg interface order [LR,RR,LF,RF], wheel targets
  clamped +-150 rad/s, obs/act delay rings (obs_delay_steps=4=80ms,
  act_delay_steps=3=60ms, ros params) with fixed negative-modulo UB
- mujoco hardware plugin: root body = free-joint body (was nonexistent
  "torso"), actuators addressed by name ({joint}_ctrl), leg torque clamp
  +-40, wheel +-5, official gas-spring force loop, 2 physics substeps per
  500 Hz tick (scene timestep 0.001), initial base z = 0.22 (absolute
  height semantics)
- bringup xacro/yaml: rear-first joint list, official gimbal scene path,
  delay params
- sim2sim defaults: obs 80 ms / act 60 ms (training-typical, measured best)
- CONTRACT.md + timing.md: authoritative values documented
- make_mjcf_from_urdf: CLI joint lists + root-body restoration (MuJoCo URDF
  import welds a jointless root to world, dropping its mass)

Note: C++ not compiled here (no ros2_control headers on this host); logic
mirrors the validated sim2sim path 1:1.

File: ros2/src/middlewares/wheeled_bringup/config/wheeled_biped.xacro (robot description, xacro)
@@ -9,5 +9,5 @@
       <xacro:if value="${'$(arg backend)' == 'sim'}">
         <plugin>wheeled_mujoco_system/WheeledMujocoSystem</plugin>
-        <param name="mjcf_path">models/wheeled_biped.xml</param>
+        <param name="mjcf_path">models/wheelbipe_v14_gimbal_scene.xml</param>
       </xacro:if>
       <xacro:if value="${'$(arg backend)' == 'real'}">
@@ -16,4 +16,16 @@
       </xacro:if>
     </hardware>
+    <!-- CONTRACT order: rear-first [LR, RR, LF, RF] (official training
+         legs_act joint order; policy obs/action dims follow this list) -->
+    <joint name="left_rear1_joint">
+      <command_interface name="position"/>
+      <state_interface name="position"/>
+      <state_interface name="velocity"/>
+    </joint>
+    <joint name="right_rear1_joint">
+      <command_interface name="position"/>
+      <state_interface name="position"/>
+      <state_interface name="velocity"/>
+    </joint>
     <joint name="left_front1_joint">
       <command_interface name="position"/>
@@ -22,14 +34,4 @@
     </joint>
     <joint name="right_front1_joint">
-      <command_interface name="position"/>
-      <state_interface name="position"/>
-      <state_interface name="velocity"/>
-    </joint>
-    <joint name="left_rear1_joint">
-      <command_interface name="position"/>
-      <state_interface name="position"/>
-      <state_interface name="velocity"/>
-    </joint>
-    <joint name="right_rear1_joint">
       <command_interface name="position"/>
       <state_interface name="position"/>
